Commit message: update

File: src/rover_autonav/description/rover.urdf.xacro (robot description, xacro)
@@ -70,5 +70,5 @@
   <xacro:wheel name="right_wheel_rear"  x="${wheelbase_rear}"    y="${-track_width/2}"/>
   <!-- ZED 2i camera mount point -->
-  <link name="zed2i_camera_link">
+  <link name="zed_camera_link">
     <visual>
       <geometry>
@@ -80,7 +80,7 @@
     </visual>
   </link>
-  <joint name="zed2i_camera_joint" type="fixed">
+  <joint name="zed_camera_joint" type="fixed">
     <parent link="base_link"/>
-    <child link="zed2i_camera_link"/>
+    <child link="zed_camera_link"/>
     <origin xyz="${camera_x} 0 ${camera_z}" rpy="0 0 0"/>
   </joint>

Commit message: rover_autonav: add full ZED TF frame chain for tracking

File: src/rover_autonav/description/rover.urdf.xacro (robot description, xacro)
@@ -13,4 +13,8 @@
   <xacro:property name="camera_x" value="0.35"/>
   <xacro:property name="camera_z" value="0.45"/>
+  <!-- ZED2i geometry constants from zed_wrapper macro -->
+  <xacro:property name="zed_height" value="0.03"/>
+  <xacro:property name="zed_baseline" value="0.12"/>
+  <xacro:property name="zed_optical_offset_x" value="-0.01"/>
   <!-- Base footprint (ground plane projection) -->
   <link name="base_footprint"/>
@@ -85,3 +89,34 @@
     <origin xyz="${camera_x} 0 ${camera_z}" rpy="0 0 0"/>
   </joint>
+  <!-- ZED frame chain required by zed_wrapper positional tracking -->
+  <link name="zed_camera_center"/>
+  <joint name="zed_camera_center_joint" type="fixed">
+    <parent link="zed_camera_link"/>
+    <child link="zed_camera_center"/>
+    <origin xyz="0 0 ${zed_height/2}" rpy="0 0 0"/>
+  </joint>
+  <link name="zed_left_camera_frame"/>
+  <joint name="zed_left_camera_joint" type="fixed">
+    <parent link="zed_camera_center"/>
+    <child link="zed_left_camera_frame"/>
+    <origin xyz="${zed_optical_offset_x} ${zed_baseline/2} 0" rpy="0 0 0"/>
+  </joint>
+  <link name="zed_left_camera_optical_frame"/>
+  <joint name="zed_left_camera_optical_joint" type="fixed">
+    <parent link="zed_left_camera_frame"/>
+    <child link="zed_left_camera_optical_frame"/>
+    <origin xyz="0 0 0" rpy="${-pi/2} 0 ${-pi/2}"/>
+  </joint>
+  <link name="zed_right_camera_frame"/>
+  <joint name="zed_right_camera_joint" type="fixed">
+    <parent link="zed_camera_center"/>
+    <child link="zed_right_camera_frame"/>
+    <origin xyz="${zed_optical_offset_x} ${-zed_baseline/2} 0" rpy="0 0 0"/>
+  </joint>
+  <link name="zed_right_camera_optical_frame"/>
+  <joint name="zed_right_camera_optical_joint" type="fixed">
+    <parent link="zed_right_camera_frame"/>
+    <child link="zed_right_camera_optical_frame"/>
+    <origin xyz="0 0 0" rpy="${-pi/2} 0 ${-pi/2}"/>
+  </joint>
 </robot>

Commit message: Update

File: src/rover_autonav/description/rover.urdf.xacro (robot description, xacro)
@@ -120,3 +120,34 @@
     <origin xyz="0 0 0" rpy="${-pi/2} 0 ${-pi/2}"/>
   </joint>
+  <!-- Compatibility aliases for zed_wrapper frame naming variants -->
+  <link name="zed_base_link"/>
+  <joint name="zed_base_link_joint" type="fixed">
+    <parent link="zed_camera_link"/>
+    <child link="zed_base_link"/>
+    <origin xyz="0 0 0" rpy="0 0 0"/>
+  </joint>
+  <link name="zed_left_camera"/>
+  <joint name="zed_left_camera_alias_joint" type="fixed">
+    <parent link="zed_left_camera_frame"/>
+    <child link="zed_left_camera"/>
+    <origin xyz="0 0 0" rpy="0 0 0"/>
+  </joint>
+  <link name="zed_left_camera_optical"/>
+  <joint name="zed_left_camera_optical_alias_joint" type="fixed">
+    <parent link="zed_left_camera_optical_frame"/>
+    <child link="zed_left_camera_optical"/>
+    <origin xyz="0 0 0" rpy="0 0 0"/>
+  </joint>
+  <link name="zed_right_camera"/>
+  <joint name="zed_right_camera_alias_joint" type="fixed">
+    <parent link="zed_right_camera_frame"/>
+    <child link="zed_right_camera"/>
+    <origin xyz="0 0 0" rpy="0 0 0"/>
+  </joint>
+  <link name="zed_right_camera_optical"/>
+  <joint name="zed_right_camera_optical_alias_joint" type="fixed">
+    <parent link="zed_right_camera_optical_frame"/>
+    <child link="zed_right_camera_optical"/>
+    <origin xyz="0 0 0" rpy="0 0 0"/>
+  </joint>
 </robot>

Commit message: Update

File: src/rover_autonav/description/rover.urdf.xacro (robot description, xacro)
@@ -151,3 +151,46 @@
     <origin xyz="0 0 0" rpy="0 0 0"/>
   </joint>
+  <!-- Extra compatibility aliases for camera-model-prefixed frame variants -->
+  <link name="zed2i_camera_link"/>
+  <joint name="zed2i_camera_link_alias_joint" type="fixed">
+    <parent link="zed_camera_link"/>
+    <child link="zed2i_camera_link"/>
+    <origin xyz="0 0 0" rpy="0 0 0"/>
+  </joint>
+  <link name="zed2i_base_link"/>
+  <joint name="zed2i_base_link_alias_joint" type="fixed">
+    <parent link="zed_base_link"/>
+    <child link="zed2i_base_link"/>
+    <origin xyz="0 0 0" rpy="0 0 0"/>
+  </joint>
+  <link name="zed2i_camera_center"/>
+  <joint name="zed2i_camera_center_alias_joint" type="fixed">
+    <parent link="zed_camera_center"/>
+    <child link="zed2i_camera_center"/>
+    <origin xyz="0 0 0" rpy="0 0 0"/>
+  </joint>
+  <link name="zed2i_left_camera_frame"/>
+  <joint name="zed2i_left_camera_frame_alias_joint" type="fixed">
+    <parent link="zed_left_camera_frame"/>
+    <child link="zed2i_left_camera_frame"/>
+    <origin xyz="0 0 0" rpy="0 0 0"/>
+  </joint>
+  <link name="zed2i_left_camera_optical_frame"/>
+  <joint name="zed2i_left_camera_optical_frame_alias_joint" type="fixed">
+    <parent link="zed_left_camera_optical_frame"/>
+    <child link="zed2i_left_camera_optical_frame"/>
+    <origin xyz="0 0 0" rpy="0 0 0"/>
+  </joint>
+  <link name="zed2i_right_camera_frame"/>
+  <joint name="zed2i_right_camera_frame_alias_joint" type="fixed">
+    <parent link="zed_right_camera_frame"/>
+    <child link="zed2i_right_camera_frame"/>
+    <origin xyz="0 0 0" rpy="0 0 0"/>
+  </joint>
+  <link name="zed2i_right_camera_optical_frame"/>
+  <joint name="zed2i_right_camera_optical_frame_alias_joint" type="fixed">
+    <parent link="zed_right_camera_optical_frame"/>
+    <child link="zed2i_right_camera_optical_frame"/>
+    <origin xyz="0 0 0" rpy="0 0 0"/>
+  </joint>
 </robot>
